File: ehrbl.kicad_pcb (KiCad board)
At the start: 2 copper layers, 234.7 x 104.6 mm, 122 parts, among them J1 3305-0-15-80-47-27-10-0, J10 3305-0-15-80-47-27-10-0, J11 3305-0-15-80-47-27-10-0, J12 3305-0-15-80-47-27-10-0, J13 3305-0-15-80-47-27-10-0, J14 3305-0-15-80-47-27-10-0, J15 3305-0-15-80-47-27-10-0, J16 3305-0-15-80-47-27-10-0, J17 3305-0-15-80-47-27-10-0, J18 3305-0-15-80-47-27-10-0, J19 3305-0-15-80-47-27-10-0, J2 3305-0-15-80-47-27-10-0, J20 3305-0-15-80-47-27-10-0, J21 3305-0-15-80-47-27-10-0, J22 3305-0-15-80-47-27-10-0, J23 3305-0-15-80-47-27-10-0, J24 3305-0-15-80-47-27-10-0, J25 3305-0-15-80-47-27-10-0, J26 3305-0-15-80-47-27-10-0, J27 3305-0-15-80-47-27-10-0, J28 3305-0-15-80-47-27-10-0, J29 3305-0-15-80-47-27-10-0, J3 3305-0-15-80-47-27-10-0, J30 3305-0-15-80-47-27-10-0, J31 3305-0-15-80-47-27-10-0, J32 3305-0-15-80-47-27-10-0, J33 3305-0-15-80-47-27-10-0, J34 3305-0-15-80-47-27-10-0, J35 3305-0-15-80-47-27-10-0, J36 3305-0-15-80-47-27-10-0, J37 3305-0-15-80-47-27-10-0, J38 3305-0-15-80-47-27-10-0, J39 3305-0-15-80-47-27-10-0, J4 3305-0-15-80-47-27-10-0, J40 3305-0-15-80-47-27-10-0, J41 3305-0-15-80-47-27-10-0, J42 3305-0-15-80-47-27-10-0, J43 3305-0-15-80-47-27-10-0, J44 3305-0-15-80-47-27-10-0, J45 3305-0-15-80-47-27-10-0, J46 3305-0-15-80-47-27-10-0, J47 3305-0-15-80-47-27-10-0, J48 3305-0-15-80-47-27-10-0, J49 3305-0-15-80-47-27-10-0, J5 3305-0-15-80-47-27-10-0, J50 3305-0-15-80-47-27-10-0, J51 3305-0-15-80-47-27-10-0, J52 3305-0-15-80-47-27-10-0, J53 MF254V-11-07-0743, J54 MF254V-11-07-0743, J55 MF254V-11-07-0743, J56 MF254V-11-07-0743, J57 0906, J58 0906, J6 3305-0-15-80-47-27-10-0, J7 3305-0-15-80-47-27-10-0, J8 3305-0-15-80-47-27-10-0, J9 3305-0-15-80-47-27-10-0, SW1 SW_Push, SW10 SW_Push, SW11 SW_Push, SW12 SW_Push, SW13 SW_Push, SW14 SW_Push, SW15 SW_Push, SW16 SW_Push, SW17 SW_Push, SW18 SW_Push, SW19 SW_Push, SW2 SW_Push, SW20 SW_Push, SW21 SW_Push, SW22 SW_Push, SW23 SW_Push, SW24 SW_Push, SW25 SW_Push, SW26 SW_Push, SW27 RotaryEncoder_Switch, SW28 RotaryEncoder_Switch, SW29 SSSS811101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

Commit message: back to 28 keys
Parts:
- removed U3, U4: MY-LR44-02, ehrbl:BAT-SMD_MY-LR44-02
- added BT1: MY-LR44-03-J, ehrbl:CONN-TH_MY-LR44-03-J, F.Cu at (232.8, 57.7)
- added BT2: MY-LR44-03-J, ehrbl:CONN-TH_MY-LR44-03-J, F.Cu at (87.1, 57.7)
- added E1: CESD5V0D3 ZA, ehrbl:SOD-323_L1.8-W1.3-LS2.5-RD, F.Cu at (245.0, 101.0)
- added E2: CESD5V0D3 ZA, ehrbl:SOD-323_L1.8-W1.3-LS2.5-RD, F.Cu at (244.5, 103.5)
- added E3: CESD5V0D3 ZA, ehrbl:SOD-323_L1.8-W1.3-LS2.5-RD, F.Cu at (250.5, 107.0)
- added E4: CESD5V0D3 ZA, ehrbl:SOD-323_L1.8-W1.3-LS2.5-RD, F.Cu at (71.5, 102.2)
- added E5: CESD5V0D3 ZA, ehrbl:SOD-323_L1.8-W1.3-LS2.5-RD, F.Cu at (69.8, 106.2)
- added E6: CESD5V0D3 ZA, ehrbl:SOD-323_L1.8-W1.3-LS2.5-RD, F.Cu at (66.8, 95.0)
- added J59: 3305-0-15-80-47-27-10-0, ehrbl:3305-0-15-80-47-27-10-0, F.Cu at (175.5, 73.1)
- added J60: 3305-0-15-80-47-27-10-0, ehrbl:3305-0-15-80-47-27-10-0, F.Cu at (170.5, 71.0)
- added J61: 3305-0-15-80-47-27-10-0, ehrbl:3305-0-15-80-47-27-10-0, F.Cu at (154.4, 73.2)
- added J62: 3305-0-15-80-47-27-10-0, ehrbl:3305-0-15-80-47-27-10-0, F.Cu at (149.4, 71.1)
- added SW31: SW_Push, ehrbl:SW_PG1350, F.Cu at (170.5, 76.9)
- added SW32: SW_Push, ehrbl:SW_PG1350, F.Cu at (149.4, 77.0)
- moved SW30 83.8 mm to (70.0, 90.9), turned to -170 degrees
- moved SW29 82.6 mm to (249.0, 90.4), turned to 170 degrees
- moved C3 80.7 mm to (67.0, 101.9), turned to -80 degrees
- moved J55 80.5 mm to (64.4, 100.3), turned to -80 degrees
- moved J58 80.4 mm to (67.5, 99.4), turned to 100 degrees
- moved J54 80.4 mm to (255.6, 100.2), turned to -100 degrees
- moved C4 80.2 mm to (67.5, 104.4), turned to -80 degrees
- moved U2 80.2 mm to (71.9, 99.0), turned to 100 degrees
- moved U1 80.1 mm to (248.0, 98.9), turned to 80 degrees
- moved J57 80.0 mm to (243.7, 97.8), turned to 80 degrees
- moved J56 79.9 mm to (79.4, 97.6), turned to -80 degrees
- moved J53 79.8 mm to (240.6, 97.5), turned to -100 degrees
- moved C1 79.0 mm to (242.5, 99.9), turned to 80 degrees
- moved C2 78.5 mm to (242.0, 102.4), turned to 80 degrees
- moved J19 12.7 mm to (213.9, 94.2)
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Connections:
- J53 pad 1: /row1 -> /col4
- J53 pad 2: /row4 -> /col3
- J53 pad 3: /row2 -> /col2
- J53 pad 4: /row3 -> /col1
- J54 pad 4: /col4 -> /row1
- J54 pad 5: /col3 -> /row2
- J54 pad 6: /col2 -> /row3
- J54 pad 7: /col1 -> /row4
- J55 pad 2: /row8 -> /row6
- J55 pad 3: /row6 -> /row7
- J55 pad 4: /row7 -> /row8
- J56 pad 4: /col8 -> /col5
- J56 pad 5: /col7 -> /col6
- J56 pad 6: /col6 -> /col7
- J56 pad 7: /col5 -> /col8
- SW29 pad 1: Net-(SW29-Pad1) -> unconnected-(SW29-Pad1)
- SW29 pad 3: unconnected-(SW29-Pad3) -> Net-(BT1-+)
- SW30 pad 1: unconnected-(SW30-Pad1) -> Net-(BT2-+)
- SW30 pad 3: Net-(SW30-Pad3) -> unconnected-(SW30-Pad3)
- U1 pad 1: /row1 -> /col4
- U1 pad 10: /col3 -> /row2
- U1 pad 11: /col4 -> /row1
- U1 pad 2: /row4 -> /col3
- U1 pad 3: /row2 -> /col2
- U1 pad 4: /row3 -> /col1
- U1 pad 8: /col1 -> /row4
- U1 pad 9: /col2 -> /row3
- U10 pad 2: /col7 -> /col6
- U10 pad 3: /sw15 -> /sw26
- U10 pad 4: /sw18 -> /sw15
- U10 pad 5: /sw26 -> /sw18
- U11 pad 2: /col6 -> /col7
- U11 pad 3: /sw16 -> unconnected-(U11-Pad3)
- U11 pad 4: /sw19 -> /sw16
- U11 pad 5: unconnected-(U11-Pad5) -> /sw19
- U12 pad 1: /sw24 -> /sw20
- U12 pad 2: /col5 -> /col8
- U12 pad 3: unconnected-(U12-Pad3) -> /sw24
- U12 pad 4: /sw20 -> unconnected-(U12-Pad4)
- U12 pad 5: unconnected-(U12-Pad5) -> /sw32
- U2 pad 10: /col7 -> /col6
- U2 pad 11: /col8 -> /col5
- U2 pad 2: /row8 -> /row6
- U2 pad 3: /row6 -> /row7
- U2 pad 4: /row7 -> /row8
- U2 pad 8: /col5 -> /col8
- U2 pad 9: /col6 -> /col7
- U5 pad 4: unconnected-(U5-Pad4) -> /sw31
- U6 pad 1: /sw5 -> unconnected-(U6-Pad1)
- U6 pad 4: unconnected-(U6-Pad4) -> /sw5
- U7 pad 1: /sw6 -> /sw12
- U7 pad 4: /sw12 -> /sw6
- U8 pad 1: /sw7 -> /sw13
- U8 pad 4: /sw13 -> /sw7
- U9 pad 2: /col8 -> /col5
- U9 pad 3: /sw14 -> /sw25
- U9 pad 4: /sw17 -> /sw14
- U9 pad 5: /sw25 -> /sw17
Routing:
- net /col1: track 20.4 -> 88.3 mm
- net /rot1a: track 101.3 -> 36.1 mm
- net /rot1b: track 96.8 -> 36.0 mm
- net Net-(SW30-Pad3): track 57.7 -> 0.00 mm
- net Net-(SW29-Pad1): track 57.4 -> 0.00 mm
- net /row4: track 146.5 -> 90.1 mm
- net /col4: track 81.4 -> 31.2 mm
- net /row8: track 134.6 -> 84.8 mm
- net /col2: track 21.4 -> 67.9 mm
- net /row5: track 69.8 -> 108.9 mm
- net /row1: track 68.2 -> 102.5 mm
- net /rot2b: track 72.0 -> 42.5 mm
- net /sw32: track 0.00 -> 29.2 mm
- net /sw31: track 0.00 -> 28.8 mm
- net /rot2a: track 72.8 -> 45.8 mm
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- added copper zone on B.Cu, net Net-(BT1-+)
- added copper zone on B.Cu, net Net-(BT2-+)
- removed copper zone on B.Cu, net GND_L
- removed copper zone on B.Cu, net GND_R
Other:
- board size 234.7 x 104.6 mm -> 234.9 x 106.1 mm
